File: kicad_project/WirelessChargerPCB.kicad_pcb (KiCad board)
At the start: 4 copper layers, 0 parts

Commit message: Agregando huellas y modelos 3D, además de otros cambios en el editor de placas y esquemático
Signed-off-by: ant0305 <anthonycalvo50@gmail.com>
Parts:
- added C1: 10uF, Capacitor_SMD:C_1206_3216Metric, F.Cu at (106.7, 84.4)
- added C2: 100nF, Capacitor_SMD:C_1206_3216Metric, F.Cu at (106.7, 90.7)
- added C3: 100nF, Capacitor_SMD:C_1206_3216Metric, F.Cu at (111.4, 78.2)
- added C4: 10nF, Capacitor_SMD:C_1206_3216Metric, F.Cu at (117.9, 78.2)
- added C5: 10nF, Capacitor_SMD:C_1206_3216Metric, F.Cu at (122.9, 83.7)
- added C6: 2nF, Capacitor_SMD:C_1206_3216Metric, F.Cu at (118.8, 95.0)
- added C7: 2nF, Capacitor_SMD:C_1206_3216Metric, F.Cu at (227.2, 86.3)
- added C8: 2.2uF, Capacitor_SMD:C_1206_3216Metric, F.Cu at (227.2, 74.8)
- added D1: 1N4148, Diode_THT:D_DO-35_SOD27_P7.62mm_Horizontal, F.Cu at (112.5, 101.1)
- added D2: 1N4148, Diode_THT:D_DO-35_SOD27_P7.62mm_Horizontal, F.Cu at (140.3, 91.4)
- added D3: SS14, Diode_SMD:D_SMA, F.Cu at (233.5, 84.9)
- added D4: SS14, Diode_SMD:D_SMA, F.Cu at (239.0, 85.0)
- added D5: SS14, Diode_SMD:D_SMA, F.Cu at (233.7, 76.5)
- added D6: SS14, Diode_SMD:D_SMA, F.Cu at (239.1, 76.5)
- added J1: Screw_Terminal_01x02, TerminalBlock:TerminalBlock_bornier-2_P5.08mm, F.Cu at (98.8, 85.0)
- added J2: Screw_Terminal_01x02, TerminalBlock:TerminalBlock_bornier-2_P5.08mm, F.Cu at (246.8, 83.5)
- added J3: Conn_01x02_Socket, Connector_PinSocket_2.54mm:PinSocket_1x02_P2.54mm_Vertical, F.Cu at (144.0, 84.1)
- added J5: Conn_01x02_Socket, Connector_PinSocket_2.54mm:PinSocket_1x02_P2.54mm_Vertical, F.Cu at (227.3, 79.3)
- added Q1: BD139, Package_TO_SOT_THT:TO-126-3_Vertical, F.Cu at (132.9, 97.5)
- added Q2: IRFZ44N, Huellas:TO254P1016X419X2286-3, F.Cu at (136.1, 78.9)
- added R1: 100Ω, Resistor_SMD:R_1206_3216Metric, F.Cu at (120.2, 100.3)
- added R2: 1kΩ, Resistor_SMD:R_1206_3216Metric, F.Cu at (123.8, 78.3)
- added R3: 150Ω, Resistor_SMD:R_1206_3216Metric, F.Cu at (122.3, 89.2)
- added REF**: MountingHole_D1.2, Huellas:MountingHole_D1.2, F.Cu at (131.5, 78.9)
- added RV1: 1kΩ, Potentiometer_THT:Potentiometer_Bourns_3296W_Vertical, F.Cu at (103.4, 77.2)
- added RV2: 1kΩ, Potentiometer_THT:Potentiometer_Bourns_3296W_Vertical, F.Cu at (98.7, 97.8)
- added U1: NE555D, Package_SO:SOIC-8_3.9x4.9mm_P1.27mm, F.Cu at (114.6, 86.9)
